Commit message: modified wpv3_rack

File: wpv3_bringup/urdf/wpv3_rack_.urdf (robot description, URDF)
Before this commit: robot WPV3_RACK, 16 links, 15 joints
Links:
- removed link rack_back
- removed link rack_beam_1
- removed link rack_beam_2
- removed link rack_beam_3
- removed link rack_beam_4
- removed link rack_level_1
- removed link rack_level_2
- removed link rack_level_3
- added link mobile_rack; visual mesh filename=package://wpv3_bringup/meshes/mobile_rack.dae scale=1 1 1
Joints:
- removed joint joint_back
- removed joint joint_beam_1
- removed joint joint_beam_2
- removed joint joint_beam_3
- removed joint joint_beam_4
- removed joint joint_level_1
- removed joint level_2
- removed joint level_3
- added joint base_rack: type fixed, parent base_link, child mobile_rack, origin xyz=0 0 0.02 rpy=0 0 3.14
- joint rack_es: origin xyz=-0.2 0 1.25 rpy=0 0 0 -> xyz=0.2 0 1.22 rpy=0 0 0; parent base_link -> mobile_rack
- joint rack_kinect2: origin xyz=0.2 0 1.26 rpy=0 0 3.14 -> xyz=-0.2 0 1.22 rpy=0 0 0; parent base_link -> mobile_rack
